File: 5V_Rail.kicad_sch (KiCad schematic)
At the start: 43 parts

Commit message: pushing the schematics works
Parts:
- C100, C102, C83, C84, C85, C86, C87, C88, C89, C90, C91, C93, C94, C96: value C -> 22u
- C101, C103, C74: value C_Polarized -> 100u
- C104, C107, C108: value C -> 1u
- C75, C76: value C -> 4.7u
- C77, C78: value C -> 100n
- C79, C80, C81, C82: value C -> 2.2u
- R14: value R -> 30k
- R15: value R -> 10k
- R16: value R -> 140K
- R17: value R -> 200K
- R18, R19, R20: value R -> 10K
- R21: value R -> 39.2K
- R22: value R -> 121K
Changed lines of the file:
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@@
 		(dnp no)
 		(fields_autoplaced yes)
-		(property "Reference" "#PWR68"
+		(property "Reference" "#PWR068"
 			(at 120.65 78.74 0)
 			(hide yes)
@@
 			(project "RF_Comput_mix"
 				(path "/68d0ebd3-4770-4e42-a15d-94722405f64d/ca568b1d-a558-4336-b7e2-be12f8fb35d1/eb9d5a69-b57b-41c2-a6cd-8f0620303a21"
-					(reference "#PWR68")
+					(reference "#PWR068")
 					(unit 1)
 				)
@@
 			)
 		)
-		(property "Value" "R"
+		(property "Value" "10K"
 			(at 234.442 100.076 90)
 			(show_name no)
@@
 			)
 		)
-		(property "Value" "C"
+		(property "Value" "22u"
 			(at 144.018 58.928 90)
 			(show_name no)
@@
 			)
 		)
-		(property "Value" "C"
+		(property "Value" "22u"
 			(at 149.098 58.928 90)
 			(show_name no)
@@
 		(in_pos_files yes)
 		(dnp no)
-		(property "Reference" "#PWR172"
+		(property "Reference" "#PWR0172"
 			(at 224.79 149.86 0)
 			(hide yes)
@@
 			(project "RF_Comput_mix"
 				(path "/68d0ebd3-4770-4e42-a15d-94722405f64d/ca568b1d-a558-4336-b7e2-be12f8fb35d1/eb9d5a69-b57b-41c2-a6cd-8f0620303a21"
-					(reference "#PWR172")
+					(reference "#PWR0172")
 					(unit 1)
 				)
@@
 			)
 		)
-		(property "Value" "C"
+		(property "Value" "100n"
 			(at 64.77 86.3601 0)
 			(show_name no)
@@
 			)
 		)
-		(property "Value" "C"
+		(property "Value" "22u"
 			(at 144.018 102.108 90)
 			(show_name no)
@@
 			)
 		)
-		(property "Value" "C"
+		(property "Value" "4.7u"
 			(at 53.594 52.832 0)
 			(show_name no)
@@
 			)
 		)
-		(property "Value" "R"
+		(property "Value" "30k"
 			(at 40.64 67.3099 0)
 			(show_name no)
@@
 			)
 		)
-		(property "Value" "C"
+		(property "Value" "22u"
 			(at 149.098 83.058 90)
 			(show_name no)
@@
 			)
 		)
-		(property "Value" "C"
+		(property "Value" "1u"
 			(at 227.33 85.852 0)
 			(show_name no)
@@
 			)
 		)
-		(property "Value" "C"
+		(property "Value" "22u"
 			(at 138.938 102.108 90)
 			(show_name no)
@@
 		(dnp no)
 		(fields_autoplaced yes)
-		(property "Reference" "#PWR193"
+		(property "Reference" "#PWR0193"
 			(at 260.35 81.28 0)
 			(hide yes)
@@
 			(project "RF_Comput_mix"
 				(path "/68d0ebd3-4770-4e42-a15d-94722405f64d/ca568b1d-a558-4336-b7e2-be12f8fb35d1/eb9d5a69-b57b-41c2-a6cd-8f0620303a21"
-					(reference "#PWR193")
+					(reference "#PWR0193")
 					(unit 1)
 				)
@@
 			)
 		)
-		(property "Value" "C"
+		(property "Value" "2.2u"
 			(at 133.858 102.108 90)
 			(show_name no)
@@
 		(dnp no)
 		(fields_autoplaced yes)
-		(property "Reference" "#PWR195"
+		(property "Reference" "#PWR0195"
 			(at 269.24 81.28 0)
 			(hide yes)
@@
 			(project "RF_Comput_mix"
 				(path "/68d0ebd3-4770-4e42-a15d-94722405f64d/ca568b1d-a558-4336-b7e2-be12f8fb35d1/eb9d5a69-b57b-41c2-a6cd-8f0620303a21"
-					(reference "#PWR195")
+					(reference "#PWR0195")
 					(unit 1)
 				)
@@
 			)
 		)
-		(property "Value" "C"
+		(property "Value" "1u"
 			(at 223.012 85.852 0)
 			(show_name no)
@@
 		(dnp no)
 		(fields_autoplaced yes)
-		(property "Reference" "#PWR192"
+		(property "Reference" "#PWR0192"
 			(at 251.46 81.28 0)
 			(hide yes)
@@
 			(project "RF_Comput_mix"
 				(path "/68d0ebd3-4770-4e42-a15d-94722405f64d/ca568b1d-a558-4336-b7e2-be12f8fb35d1/eb9d5a69-b57b-41c2-a6cd-8f0620303a21"
-					(reference "#PWR192")
+					(reference "#PWR0192")
 					(unit 1)
 				)
@@
 			)
 		)
-		(property "Value" "R"
+		(property "Value" "10K"
 			(at 234.442 103.886 90)
 			(show_name no)
@@
 			)
 		)
-		(property "Value" "C"
+		(property "Value" "100n"
 			(at 60.452 53.086 0)
 			(show_name no)
@@
 		(dnp no)
 		(fields_autoplaced yes)
-		(property "Reference" "#PWR169"
+		(property "Reference" "#PWR0169"
 			(at 218.44 93.98 0)
 			(hide yes)
@@
 			(project "RF_Comput_mix"
 				(path "/68d0ebd3-4770-4e42-a15d-94722405f64d/ca568b1d-a558-4336-b7e2-be12f8fb35d1/eb9d5a69-b57b-41c2-a6cd-8f0620303a21"
-					(reference "#PWR169")
+					(reference "#PWR0169")
 					(unit 1)
 				)
@@
 			)
 		)
-		(property "Value" "R"
+		(property "Value" "39.2K"
 			(at 256.032 71.882 0)
 			(show_name no)
@@
 			)
 		)
-		(property "Value" "C"
+		(property "Value" "22u"
 			(at 138.938 46.228 90)
 			(show_name no)
@@
 		(in_pos_files yes)
 		(dnp no)
-		(property "Reference" "#PWR170"
+		(property "Reference" "#PWR0170"
 			(at 224.79 128.27 0)
 			(hide yes)
@@
 			(project "RF_Comput_mix"
 				(path "/68d0ebd3-4770-4e42-a15d-94722405f64d/ca568b1d-a558-4336-b7e2-be12f8fb35d1/eb9d5a69-b57b-41c2-a6cd-8f0620303a21"
-					(reference "#PWR170")
+					(reference "#PWR0170")
 					(unit 1)
 				)
@@
 			)
 		)
-		(property "Value" "C"
+		(property "Value" "22u"
 			(at 144.018 83.058 90)
 			(show_name no)
@@
 			)
 		)
-		(property "Value" "C"
+		(property "Value" "22u"
 			(at 138.938 83.058 90)
 			(show_name no)
@@
 		(in_pos_files yes)
 		(dnp no)
-		(property "Reference" "#PWR188"
+		(property "Reference" "#PWR0188"
 			(at 233.68 93.98 0)
 			(hide yes)
@@
 			(project "RF_Comput_mix"
 				(path "/68d0ebd3-4770-4e42-a15d-94722405f64d/ca568b1d-a558-4336-b7e2-be12f8fb35d1/eb9d5a69-b57b-41c2-a6cd-8f0620303a21"
-					(reference "#PWR188")
+					(reference "#PWR0188")
 					(unit 1)
 				)
@@
 			)
 		)
-		(property "Value" "C"
+		(property "Value" "22u"
 			(at 149.098 102.108 90)
 			(show_name no)
@@
 			)
 		)
-		(property "Value" "R"
+		(property "Value" "140K"
 			(at 64.77 63.246 0)
 			(show_name no)
@@
 		(in_pos_files yes)
 		(dnp no)
-		(property "Reference" "#PWR58"
+		(property "Reference" "#PWR058"
 			(at 68.58 69.85 0)
 			(hide yes)
@@
 			(project "RF_Comput_mix"
 				(path "/68d0ebd3-4770-4e42-a15d-94722405f64d/ca568b1d-a558-4336-b7e2-be12f8fb35d1/eb9d5a69-b57b-41c2-a6cd-8f0620303a21"
-					(reference "#PWR58")
+					(reference "#PWR058")
 					(unit 1)
 				)
@@
 			)
 		)
-		(property "Value" "C"
+		(property "Value" "1u"
 			(at 234.95 86.106 0)
 			(show_name no)
@@
 			)
 		)
-		(property "Value" "C"
+		(property "Value" "4.7u"
 			(at 53.086 88.9 0)
 			(show_name no)
@@
 			)
 		)
-		(property "Value" "C"
+		(property "Value" "22u"
 			(at 154.178 46.228 90)
 			(show_name no)
@@
 			)
 		)
-		(property "Value" "C"
+		(property "Value" "2.2u"
 			(at 133.858 83.058 90)
 			(show_name no)
@@
 			)
 		)
-		(property "Value" "C_Polarized"
+		(property "Value" "100u"
 			(at 154.178 103.378 90)
 			(show_name no)
@@
 			)
 		)
-		(property "Value" "R"
+		(property "Value" "10K"
 			(at 248.158 71.882 0)
 			(show_name no)
@@
 			)
 		)
-		(property "Value" "R"
+		(property "Value" "121K"
 			(at 264.922 71.882 0)
 			(show_name no)
@@
 			)
 		)
-		(property "Value" "C_Polarized"
+		(property "Value" "100u"
 			(at 43.434 53.594 0)
 			(show_name no)
@@
 			)
 		)
-		(property "Value" "C"
+		(property "Value" "22u"
 			(at 149.098 46.228 90)
 			(show_name no)
@@
 			)
 		)
-		(property "Value" "C"
+		(property "Value" "22u"
 			(at 144.018 46.228 90)
 			(show_name no)
@@
 		(in_pos_files yes)
 		(dnp no)
-		(property "Reference" "#PWR171"
+		(property "Reference" "#PWR0171"
 			(at 224.79 138.43 0)
 			(hide yes)
@@
 			(project "RF_Comput_mix"
 				(path "/68d0ebd3-4770-4e42-a15d-94722405f64d/ca568b1d-a558-4336-b7e2-be12f8fb35d1/eb9d5a69-b57b-41c2-a6cd-8f0620303a21"
-					(reference "#PWR171")
+					(reference "#PWR0171")
 					(unit 1)
 				)
@@
 			)
 		)
-		(property "Value" "R"
+		(property "Value" "10k"
 			(at 40.64 74.9299 0)
 			(show_name no)
@@
 			)
 		)
-		(property "Value" "R"
+		(property "Value" "200K"
 			(at 116.84 70.358 0)
 			(show_name no)
@@
 			)
 		)
-		(property "Value" "C"
+		(property "Value" "22u"
 			(at 154.178 83.058 90)
 			(show_name no)
@@
 			)
 		)
-		(property "Value" "C"
+		(property "Value" "2.2u"
 			(at 133.858 46.228 90)
 			(show_name no)
@@
 			)
 		)
-		(property "Value" "C"
+		(property "Value" "2.2u"
 			(at 133.858 58.928 90)
 			(show_name no)
@@
 			)
 		)
-		(property "Value" "C_Polarized"
+		(property "Value" "100u"
 			(at 154.178 60.198 90)
 			(show_name no)
@@
 			)
 		)
-		(property "Value" "C"
+		(property "Value" "22u"
 			(at 138.938 58.928 90)
 			(show_name no)
