File: Bank67.kicad_sch (KiCad schematic)
At the start: 2 parts, among them U1 XCKU5P-FFVB676

Commit message: pushing the schematics works
Parts:
- removed R63: R, Resistor_SMD:R_0201_0603Metric, symbol Device:R
- added R48: 240, Resistor_SMD:R_0201_0603Metric, symbol Device:R
Connections:
- net GND: now also R48.2
- net VRP: now also R48.1
- net IO_L10N_T1U_N7_QBC_AD4N_67_N renamed D4a.UDQS_c
- net IO_L10P_T1U_N6_QBC_AD4P_67_P renamed D4a.UDQS_t
- net IO_L11N_T1U_N9_GC_67_N renamed D4b_DQ13
- net IO_L11P_T1U_N8_GC_67_P renamed D4b_DQ12
- net IO_L12N_T1U_N11_GC_67_N renamed D4b_DQ15
- net IO_L12P_T1U_N10_GC_67_P renamed D4b_DQ14
- net IO_L13N_T2L_N1_GC_QBC_67_N: no longer names the net of U1.C19 (IO_L13N_T2L_N1_GC_QBC_67_N)
- net IO_L13P_T2L_N0_GC_QBC_67_P renamed D4b.~{LDBI}
- net IO_L14N_T2L_N3_GC_67_N renamed D4a_DQ1
- net IO_L14P_T2L_N2_GC_67_P renamed D4a_DQ0
- net IO_L15N_T2L_N5_AD11N_67_N renamed D4a_DQ3
- net IO_L15P_T2L_N4_AD11P_67_P renamed D4a_DQ2
- net IO_L16N_T2U_N7_QBC_AD3N_67_N renamed D4b.LDQS_c
- net IO_L16P_T2U_N6_QBC_AD3P_67_P renamed D4b.LDQS_t
- net IO_L17N_T2U_N9_AD10N_67_N renamed D4a_DQ5
- net IO_L17P_T2U_N8_AD10P_67_P renamed D4a_DQ4
- net IO_L18N_T2U_N11_AD2N_67_N renamed D4a_DQ7
- net IO_L18P_T2U_N10_AD2P_67_P renamed D4a_DQ6
- net IO_L19N_T3L_N1_DBC_AD9N_67_N: no longer names the net of U1.A23 (IO_L19N_T3L_N1_DBC_AD9N_67_N)
- net IO_L19P_T3L_N0_DBC_AD9P_67_P renamed D4b.~{UDBI}
- net IO_L1N_T0L_N1_DBC_67_N: no longer names the net of U1.F15 (IO_L1N_T0L_N1_DBC_67_N)
- net IO_L1P_T0L_N0_DBC_67_P renamed D4a.~{LDBI}
- net IO_L20N_T3L_N3_AD1N_67_N renamed D4a_DQ9
- net IO_L20P_T3L_N2_AD1P_67_P renamed D4a_DQ8
- net IO_L21N_T3L_N5_AD8N_67_N renamed D4a_DQ11
- net IO_L21P_T3L_N4_AD8P_67_P renamed D4a_DQ10
- net IO_L22N_T3U_N7_DBC_AD0N_67_N renamed D4b.UDQS_c
- net IO_L22P_T3U_N6_DBC_AD0P_67_P renamed D4b.UDQS_t
- net IO_L23N_T3U_N9_67_N renamed D4a_DQ13
- net IO_L23P_T3U_N8_67_P renamed D4a_DQ12
- net IO_L24N_T3U_N11_67_N renamed D4a_DQ15
- net IO_L24P_T3U_N10_67_P renamed D4a_DQ14
- net IO_L2N_T0L_N3_67_N renamed D4b_DQ1
- net IO_L2P_T0L_N2_67_P renamed D4b_DQ0
- net IO_L3N_T0L_N5_AD15N_67_N renamed D4b_DQ3
- net IO_L3P_T0L_N4_AD15P_67_P renamed D4b_DQ2
- net IO_L4N_T0U_N7_DBC_AD7N_67_N renamed D4a.LDQS_c
- net IO_L4P_T0U_N6_DBC_AD7P_67_P renamed D4a.LDQS_t
- net IO_L5N_T0U_N9_AD14N_67_N renamed D4b_DQ5
- net IO_L5P_T0U_N8_AD14P_67_P renamed D4b_DQ4
- net IO_L6N_T0U_N11_AD6N_67_N renamed D4b_DQ7
- net IO_L6P_T0U_N10_AD6P_67_P renamed D4b_DQ6
- net IO_L7N_T1L_N1_QBC_AD13N_67_N: no longer names the net of U1.H19 (IO_L7N_T1L_N1_QBC_AD13N_67_N)
- net IO_L7P_T1L_N0_QBC_AD13P_67_P renamed D4a.~{UDBI}
- net IO_L8N_T1L_N3_AD5N_67_N renamed D4b_DQ9
- net IO_L8P_T1L_N2_AD5P_67_P renamed D4b_DQ8
- net IO_L9N_T1L_N5_AD12N_67_N renamed D4b_DQ11
- net IO_L9P_T1L_N4_AD12P_67_P renamed D4b_DQ10
- net IO_T1U_N12_67: no longer names the net of U1.G19 (IO_T1U_N12_67)
- net IO_T2U_N12_67: no longer names the net of U1.B16 (IO_T2U_N12_67)
- net IO_T3U_N12_67: no longer names the net of U1.E22 (IO_T3U_N12_67)
