File: DDR4.kicad_sch (KiCad schematic)
At the start: 13 parts, among them U2 MT40A512M16TB, U4 MT40A512M16TB

Commit message: pushing the schematics works
Parts:
- C175, C176: value C -> 100n
- R31, R32: value R -> 1k
- R33, R34, R37, R38: value R -> 10k
- R35: value R -> 4.7k
- R39, R40: value R -> 240
Changed lines of the file:
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@@
 			)
 		)
-		(property "Value" "R"
+		(property "Value" "240"
 			(at 128.27 149.8599 0)
 			(show_name no)
@@
 			)
 		)
-		(property "Value" "R"
+		(property "Value" "10k"
 			(at 182.88 134.6199 0)
 			(show_name no)
@@
 			)
 		)
-		(property "Value" "R"
+		(property "Value" "10k"
 			(at 140.97 135.8899 0)
 			(show_name no)
@@
 			)
 		)
-		(property "Value" "R"
+		(property "Value" "1k"
 			(at 267.97 146.0499 0)
 			(show_name no)
@@
 			)
 		)
-		(property "Value" "R"
+		(property "Value" "4.7k"
 			(at 259.588 129.54 0)
 			(show_name no)
@@
 			)
 		)
-		(property "Value" "R"
+		(property "Value" "1k"
 			(at 267.97 132.0799 0)
 			(show_name no)
@@
 			)
 		)
-		(property "Value" "R"
+		(property "Value" "10k"
 			(at 55.88 134.6199 0)
 			(show_name no)
@@
 			)
 		)
-		(property "Value" "C"
+		(property "Value" "100n"
 			(at 148.082 147.066 0)
 			(show_name no)
@@
 			)
 		)
-		(property "Value" "C"
+		(property "Value" "100n"
 			(at 275.082 147.066 0)
 			(show_name no)
@@
 			)
 		)
-		(property "Value" "R"
+		(property "Value" "240"
 			(at 255.27 149.8599 0)
 			(show_name no)
@@
 			)
 		)
-		(property "Value" "R"
+		(property "Value" "10k"
 			(at 140.97 146.0499 0)
 			(show_name no)
