File: DDR4_TERM.kicad_sch (KiCad schematic)
At the start: 35 parts

Commit message: pushing the schematics works
Parts:
- C177, C178, C179, C180, C181, C182, C183, C184, C185, C186, C187, C188, C189, C190, C191, C192, C193, C222, C223, C224, C225, C226, C227, C228, C229, C230: value C -> 100n
- C231: value C -> 10n
- R41: value R -> 10k
- RN1, RN2, RN3, RN4, RN5, RN6, RN7: value R_Pack04 -> 39ohm
Changed lines of the file:
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@@
 			)
 		)
-		(property "Value" "C"
+		(property "Value" "100n"
 			(at 169.672 136.906 0)
 			(show_name no)
@@
 			)
 		)
-		(property "Value" "R_Pack04"
+		(property "Value" "39ohm"
 			(at 226.06 35.5599 0)
 			(show_name no)
@@
 			)
 		)
-		(property "Value" "R_Pack04"
+		(property "Value" "39ohm"
 			(at 207.01 35.5599 0)
 			(show_name no)
@@
 			)
 		)
-		(property "Value" "C"
+		(property "Value" "100n"
 			(at 151.892 136.906 0)
 			(show_name no)
@@
 			)
 		)
-		(property "Value" "R_Pack04"
+		(property "Value" "39ohm"
 			(at 187.96 35.5599 0)
 			(show_name no)
@@
 			)
 		)
-		(property "Value" "R"
+		(property "Value" "10k"
 			(at 100.33 149.8599 0)
 			(show_name no)
@@
 			)
 		)
-		(property "Value" "R_Pack04"
+		(property "Value" "39ohm"
 			(at 168.91 35.5599 0)
 			(show_name no)
@@
 			)
 		)
-		(property "Value" "C"
+		(property "Value" "100n"
 			(at 143.002 136.906 0)
 			(show_name no)
@@
 			)
 		)
-		(property "Value" "C"
+		(property "Value" "100n"
 			(at 219.202 145.796 0)
 			(show_name no)
@@
 			)
 		)
-		(property "Value" "C"
+		(property "Value" "100n"
 			(at 158.242 145.796 0)
 			(show_name no)
@@
 			)
 		)
-		(property "Value" "C"
+		(property "Value" "100n"
 			(at 221.742 136.906 0)
 			(show_name no)
@@
 			)
 		)
-		(property "Value" "C"
+		(property "Value" "100n"
 			(at 201.422 145.796 0)
 			(show_name no)
@@
 			)
 		)
-		(property "Value" "C"
+		(property "Value" "100n"
 			(at 212.852 136.906 0)
 			(show_name no)
@@
 			)
 		)
-		(property "Value" "C"
+		(property "Value" "100n"
 			(at 210.312 145.796 0)
 			(show_name no)
@@
 			)
 		)
-		(property "Value" "C"
+		(property "Value" "100n"
 			(at 160.782 136.906 0)
 			(show_name no)
@@
 			)
 		)
-		(property "Value" "C"
+		(property "Value" "100n"
 			(at 186.182 136.906 0)
 			(show_name no)
@@
 			)
 		)
-		(property "Value" "C"
+		(property "Value" "100n"
 			(at 122.682 145.796 0)
 			(show_name no)
@@
 			)
 		)
-		(property "Value" "C"
+		(property "Value" "100n"
 			(at 113.792 145.796 0)
 			(show_name no)
@@
 			)
 		)
-		(property "Value" "C"
+		(property "Value" "100n"
 			(at 131.572 145.796 0)
 			(show_name no)
@@
 			)
 		)
-		(property "Value" "C"
+		(property "Value" "100n"
 			(at 116.332 136.906 0)
 			(show_name no)
@@
 			)
 		)
-		(property "Value" "C"
+		(property "Value" "10n"
 			(at 242.062 26.416 0)
 			(show_name no)
@@
 			)
 		)
-		(property "Value" "C"
+		(property "Value" "100n"
 			(at 134.112 136.906 0)
 			(show_name no)
@@
 			)
 		)
-		(property "Value" "C"
+		(property "Value" "100n"
 			(at 192.532 145.796 0)
 			(show_name no)
@@
 			)
 		)
-		(property "Value" "R_Pack04"
+		(property "Value" "39ohm"
 			(at 246.38 35.5599 0)
 			(show_name no)
@@
 			)
 		)
-		(property "Value" "C"
+		(property "Value" "100n"
 			(at 176.022 145.796 0)
 			(show_name no)
@@
 			)
 		)
-		(property "Value" "C"
+		(property "Value" "100n"
 			(at 178.562 136.906 0)
 			(show_name no)
@@
 			)
 		)
-		(property "Value" "R_Pack04"
+		(property "Value" "39ohm"
 			(at 130.81 35.5599 0)
 			(show_name no)
@@
 			)
 		)
-		(property "Value" "C"
+		(property "Value" "100n"
 			(at 107.442 136.906 0)
 			(show_name no)
@@
 			)
 		)
-		(property "Value" "C"
+		(property "Value" "100n"
 			(at 167.132 145.796 0)
 			(show_name no)
@@
 			)
 		)
-		(property "Value" "C"
+		(property "Value" "100n"
 			(at 140.462 145.796 0)
 			(show_name no)
@@
 			)
 		)
-		(property "Value" "R_Pack04"
+		(property "Value" "39ohm"
 			(at 149.86 35.5599 0)
 			(show_name no)
@@
 			)
 		)
-		(property "Value" "C"
+		(property "Value" "100n"
 			(at 195.072 136.906 0)
 			(show_name no)
@@
 			)
 		)
-		(property "Value" "C"
+		(property "Value" "100n"
 			(at 125.222 136.906 0)
 			(show_name no)
@@
 			)
 		)
-		(property "Value" "C"
+		(property "Value" "100n"
 			(at 149.352 145.796 0)
 			(show_name no)
@@
 			)
 		)
-		(property "Value" "C"
+		(property "Value" "100n"
 			(at 203.962 136.906 0)
 			(show_name no)
