File: Decap.kicad_sch (KiCad schematic)
At the start: 37 parts

Commit message: pushing the schematics works
Parts:
- C133, C155: value C -> 330u
- C134, C156, C157, C158: value C -> 100u
- C135, C147, C148, C149, C150, C151, C152, C153, C154, C159, C163: value C -> 47u
- C136, C140, C141, C142, C143, C144, C145, C146, C160, C161, C162, C164, C171: value C -> 10u
- C137, C138, C139: value C -> 4.7u
- C165, C166, C167, C168: value C -> 100n
Changed lines of the file:
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@@
 			)
 		)
-		(property "Value" "C"
+		(property "Value" "100u"
 			(at 148.082 49.276 0)
 			(show_name no)
@@
 			)
 		)
-		(property "Value" "C"
+		(property "Value" "10u"
 			(at 259.588 35.306 0)
 			(show_name no)
@@
 			)
 		)
-		(property "Value" "C"
+		(property "Value" "100n"
 			(at 239.522 64.516 0)
 			(show_name no)
@@
 			)
 		)
-		(property "Value" "C"
+		(property "Value" "47u"
 			(at 160.782 63.246 0)
 			(show_name no)
@@
 			)
 		)
-		(property "Value" "C"
+		(property "Value" "330u"
 			(at 148.082 34.036 0)
 			(show_name no)
@@
 			)
 		)
-		(property "Value" "C"
+		(property "Value" "47u"
 			(at 184.912 64.516 0)
 			(show_name no)
@@
 			)
 		)
-		(property "Value" "C"
+		(property "Value" "10u"
 			(at 201.422 64.516 0)
 			(show_name no)
@@
 			)
 		)
-		(property "Value" "C"
+		(property "Value" "10u"
 			(at 148.082 77.216 0)
 			(show_name no)
@@
 			)
 		)
-		(property "Value" "C"
+		(property "Value" "100u"
 			(at 141.732 49.276 0)
 			(show_name no)
@@
 			)
 		)
-		(property "Value" "C"
+		(property "Value" "47u"
 			(at 253.238 35.306 0)
 			(show_name no)
@@
 			)
 		)
-		(property "Value" "C"
+		(property "Value" "10u"
 			(at 154.432 77.216 0)
 			(show_name no)
@@
 			)
 		)
-		(property "Value" "C"
+		(property "Value" "47u"
 			(at 154.432 63.246 0)
 			(show_name no)
@@
 			)
 		)
-		(property "Value" "C"
+		(property "Value" "100n"
 			(at 207.772 64.516 0)
 			(show_name no)
@@
 			)
 		)
-		(property "Value" "C"
+		(property "Value" "10u"
 			(at 244.348 35.306 0)
 			(show_name no)
@@
 			)
 		)
-		(property "Value" "C"
+		(property "Value" "4.7u"
 			(at 206.502 35.306 0)
 			(show_name no)
@@
 			)
 		)
-		(property "Value" "C"
+		(property "Value" "47u"
 			(at 148.082 63.246 0)
 			(show_name no)
@@
 			)
 		)
-		(property "Value" "C"
+		(property "Value" "10u"
 			(at 141.732 77.216 0)
 			(show_name no)
@@
 			)
 		)
-		(property "Value" "C"
+		(property "Value" "10u"
 			(at 167.132 77.216 0)
 			(show_name no)
@@
 			)
 		)
-		(property "Value" "C"
+		(property "Value" "4.7u"
 			(at 184.912 35.306 0)
 			(show_name no)
@@
 			)
 		)
-		(property "Value" "C"
+		(property "Value" "330u"
 			(at 141.732 34.036 0)
 			(show_name no)
@@
 			)
 		)
-		(property "Value" "C"
+		(property "Value" "47u"
 			(at 223.012 35.56 0)
 			(show_name no)
@@
 			)
 		)
-		(property "Value" "C"
+		(property "Value" "10u"
 			(at 160.782 77.216 0)
 			(show_name no)
@@
 			)
 		)
-		(property "Value" "C"
+		(property "Value" "4.7u"
 			(at 196.342 35.306 0)
 			(show_name no)
@@
 			)
 		)
-		(property "Value" "C"
+		(property "Value" "47u"
 			(at 251.968 64.516 0)
 			(show_name no)
@@
 			)
 		)
-		(property "Value" "C"
+		(property "Value" "10u"
 			(at 229.362 35.56 0)
 			(show_name no)
@@
 			)
 		)
-		(property "Value" "C"
+		(property "Value" "100u"
 			(at 160.782 49.276 0)
 			(show_name no)
@@
 			)
 		)
-		(property "Value" "C"
+		(property "Value" "10u"
 			(at 214.122 64.516 0)
 			(show_name no)
@@
 			)
 		)
-		(property "Value" "C"
+		(property "Value" "47u"
 			(at 167.132 63.246 0)
 			(show_name no)
@@
 			)
 		)
-		(property "Value" "C"
+		(property "Value" "47u"
 			(at 216.662 35.56 0)
 			(show_name no)
@@
 			)
 		)
-		(property "Value" "C"
+		(property "Value" "47u"
 			(at 141.732 63.246 0)
 			(show_name no)
@@
 			)
 		)
-		(property "Value" "C"
+		(property "Value" "47u"
 			(at 237.998 35.306 0)
 			(show_name no)
@@
 			)
 		)
-		(property "Value" "C"
+		(property "Value" "100n"
 			(at 258.572 64.516 0)
 			(show_name no)
@@
 			)
 		)
-		(property "Value" "C"
+		(property "Value" "10u"
 			(at 232.918 64.516 0)
 			(show_name no)
@@
 			)
 		)
-		(property "Value" "C"
+		(property "Value" "10u"
 			(at 191.262 64.516 0)
 			(show_name no)
@@
 			)
 		)
-		(property "Value" "C"
+		(property "Value" "100n"
 			(at 220.472 64.516 0)
 			(show_name no)
@@
 			)
 		)
-		(property "Value" "C"
+		(property "Value" "10u"
 			(at 173.482 77.216 0)
 			(show_name no)
@@
 			)
 		)
-		(property "Value" "C"
+		(property "Value" "100u"
 			(at 154.432 49.276 0)
 			(show_name no)
