File: FAN.kicad_sch (KiCad schematic)
At the start: 6 parts, among them J4 Conn_01x02_Pin, M1 Fan_4pin, Q1 DMN2041L

Commit message: pushing the schematics works
Parts:
- removed C106: C_Polarized, Capacitor_Tantalum_SMD:CP_EIA-7343-31_Kemet-D, symbol Device:C_Polarized
- removed J4: Conn_01x02_Pin, Connector_JST:JST_XA_B02B-XASK-1_1x02_P2.50mm_Vertical, symbol Connector:Conn_01x02_Pin
- C73, M1, Q1, R45: now fitted; now in the parts list
Connections:
- net Tacho: now reaches M1.3 (Tacho)
- net PWM: now reaches M1.4 (PWM), Q1.3 (D)
- no-connect marks 1 -> 0
