File: FPGA_Power.kicad_sch (KiCad schematic)
At the start: 20 parts, among them U1 XCKU5P-FFVB676

Commit message: pushing the schematics works
Parts:
- C170, C174: value C -> 4.7u
- C232, C235, C236, C237, C238: value C -> 100n
- FB1: value FerriteBead_Small -> 120@100MHz
- FB2: value FerriteBead_Small -> 600@100MHz
- R13, R23, R25, R26, R27, R28, R29, R30: value R -> 1k
- R46: value R -> 100
