File: FPGA_SYS.kicad_sch (KiCad schematic)
At the start: 19 parts, among them J1 Conn_01x06_MountingPin, J2 Conn_01x02_MountingPin, SW1 SW_DIP_x03, SW2 SW_Push, U1 XCKU5P-FFVB676, U5 TXB0106RGY, U6 GD25QxxxEY

Commit message: pushing the schematics works
Parts:
- C169: value C -> 4.7u
- C173, C233, C241, C242: value C -> 100n
- D2: value LED -> Green
- J1: value Conn_01x06_MountingPin -> GH1.25 6P
- J2: value Conn_01x02_MountingPin -> GH1.25_2P
- R36: value R -> 0
- R42, R43: value R -> 20.5K
- R44: value R -> 4.7K
- RN8: value R_Pack04 -> 10k
- SW2: value SW_Push -> 6x3.6
- U6: value GD25QxxxEY -> GD25LB256
Other:
- moved on the sheet: C169, C173, U6
