File: GTY.kicad_sch (KiCad schematic)
At the start: 1 part, among them U1 XCKU5P-FFVB676

Commit message: pushing the schematics works
Parts:
- added C403, C404, C405, C406, C407, C408, C409, C410, C411, C412, C413, C414, C415, C416, C417, C418, C419, C420, C421, C422, C423, C424: 100n, Capacitor_SMD:C_0201_0603Metric, symbol Device:C
Connections:
- net MGTYTXN0_226_N: now also C404.1
- net MGTYTXN0_227_N: now also C412.1
- net MGTYTXN1_226_N: now also C406.1
- net MGTYTXN1_227_N: now also C414.1
- net MGTYTXN2_226_N: now also C408.1
- net MGTYTXN2_227_N: now also C416.1
- net MGTYTXN3_226_N: now also C410.1
- net MGTYTXP0_226_P: now also C403.1
- net MGTYTXP0_227_P: now also C411.1
- net MGTYTXP1_226_P: now also C405.1
- net MGTYTXP1_227_P: now also C413.1
- net MGTYTXP2_226_P: now also C407.1
- net MGTYTXP2_227_P: now also C415.1
- net MGTYTXP3_226_P: now also C409.1
- net SERDINA+: now also C417.2; no longer U1.AF7 (MGTYTXP0_224_P)
- net SERDINA-: now also C418.2; no longer U1.AF6 (MGTYTXN0_224_N)
- net SERDINB+: now also C419.2; no longer U1.AE9 (MGTYTXP1_224_P)
- net SERDINB-: now also C420.2; no longer U1.AE8 (MGTYTXN1_224_N)
- net SERDINC+: now also C421.2; no longer U1.AD7 (MGTYTXP2_224_P)
- net SERDINC-: now also C422.2; no longer U1.AD6 (MGTYTXN2_224_N)
- net SERDIND+: now also C423.2; no longer U1.AC5 (MGTYTXP3_224_P)
- net SERDIND-: now also C424.2; no longer U1.AC4 (MGTYTXN3_224_N)
- net MGTREFCLK1N_224_N renamed GTY_DEVCLK-
- net MGTREFCLK1N_226_N renamed PCIE0_REFCLK_N
- net MGTREFCLK1N_227_N renamed PCIE3_REFCLK_N
- net MGTREFCLK1P_224_P renamed GTY_DEVCLK+
- net MGTREFCLK1P_226_P renamed PCIE0_REFCLK_P
- net MGTREFCLK1P_227_P renamed PCIE3_REFCLK_P
- new net MGTYTXN0_224_N: C418.1, U1.AF6 (MGTYTXN0_224_N)
- new net MGTYTXN1_224_N: C420.1, U1.AE8 (MGTYTXN1_224_N)
- new net MGTYTXN2_224_N: C422.1, U1.AD6 (MGTYTXN2_224_N)
- new net MGTYTXN3_224_N: C424.1, U1.AC4 (MGTYTXN3_224_N)
- new net MGTYTXP0_224_P: C417.1, U1.AF7 (MGTYTXP0_224_P)
- new net MGTYTXP1_224_P: C419.1, U1.AE9 (MGTYTXP1_224_P)
- new net MGTYTXP2_224_P: C421.1, U1.AD7 (MGTYTXP2_224_P)
- new net MGTYTXP3_224_P: C423.1, U1.AC5 (MGTYTXP3_224_P)
- new net PCIE0_RX0N: C403.2
- new net PCIE0_RX0P: C404.2
- new net PCIE0_RX1N: C405.2
- new net PCIE0_RX1P: C406.2
- new net PCIE0_RX2N: C407.2
- new net PCIE0_RX2P: C408.2
- new net PCIE0_RX3N: C409.2
- new net PCIE0_RX3P: C410.2
- new net PCIE1_RX0N: C411.2
- new net PCIE1_RX0P: C412.2
- new net PCIE2_RX0_N: C415.2
- new net PCIE2_RX0_P: C416.2
- new net PCIE2_RX1_N: C413.2
- new net PCIE2_RX1_P: C414.2
Other:
- note added: "JESD204 TX/RX mark from ADRV9026"
- note added: "PCIE have inverted diff pair TX/RX mark from host device"
- moved on the sheet: U1A
