File: Power.kicad_sch (KiCad schematic)
At the start: 6 parts, among them SW3 SW_Push, U3 LP5912-1.5DRV

Commit message: pushing the schematics works
Parts:
- BT1: value Battery -> MS621F
- C234: value C -> 100n
- C269, C99: value C -> 1u
- SW3: value SW_Push -> 6x3.6
- U3: footprint Package_SON:WSON-6-1EP_2x2mm_P0.65mm_EP1x1.6mm_ThermalVias -> Package_SON:WSON-6-1EP_2x2mm_P0.65mm_EP1x1.6mm
