File: RF_DCDC.kicad_sch (KiCad schematic)
At the start: 60 parts

Commit message: pushing the schematics works
Parts:
- C116, C256, C258: value C_Polarized -> 100u
- C117, C118: value C -> 4.7u
- C119, C120: value C -> 100n
- C121, C122, C123, C124: value C -> 2.2u
- C125, C126, C127, C128, C129, C130, C131, C132, C172, C239, C240, C243, C244, C245, C253, C254, C255, C257, C271, C272, C273, C274, C275, C276, C277, C278, C279, C280, C281, C282: value C -> 22u
- C259, C260, C261: value C -> 1u
- R59: value R -> 69.8K
- R60, R66: value R -> 121K
- R61: value R -> 140K
- R62: value R -> 10K
- R64: value R -> 39.2K
- R65: value R -> 180K
- R77, R78: value R -> 100K
