File: RF_LDO.kicad_sch (KiCad schematic)
At the start: 40 parts, among them U10 TPS7A94, U11 TPS7A94, U8 TPS7A94, U9 TPS7A94

Commit message: pushing the schematics works
Parts:
- C109, C110, C111, C112, C113, C262, C264, C266, C268: value C -> 10u
- C114, C115, C265, C270: value C -> 1u
- C263, C267: value C -> 4.7u
- FB3, FB4, FB5, FB6: value FerriteBead_Small -> 120ohm@100MHz
- R51, R52, R67, R71: value R -> 100k
- R53: value R -> 4.32k
- R55, R57: value R -> 68.1k
- R56, R58, R70, R74: value R -> 12.4k
- R68: value R -> 6.65k
- R69: value R -> 49.3k
- R72: value R -> 12k
- R73: value R -> 98.8k
- R75, R76: value R -> 200
