File: RF_SERDES.kicad_sch (KiCad schematic)
At the start: 4 parts, among them U12 ADRV9026BBCZ

Commit message: pushing the schematics works
Parts:
- removed NT23, NT24: NetTie_2, NetTie:NetTie-2_SMD_Pad2.0mm, symbol Device:NetTie_2
- removed R79: 4.99k, Resistor_SMD:R_0201_0603Metric, symbol Device:R
- removed U12: ADRV9026BBCZ, Package_BGA:LFBGA-289_14x14mm_Layout17x17_P0.8mm, symbol dfdtc_RF:ADRV9026BBCZ
- added C425, C426, C427, C428, C429, C430, C431, C432: 100n, Capacitor_SMD:C_0201_0603Metric, symbol Device:C
- added R87: 100, Resistor_SMD:R_0201_0603Metric, symbol Device:R
- added U12: ADRV9026BBCZ, Package_BGA:LFBGA-289_14x14mm_Layout17x17_P0.8mm, symbol dfdtc_RF:ADRV9026BBCZ
Connections:
- new net DEVCLK+: R87.1, U12.C8 (DEVCLK+)
- new net DEVCLK-: R87.2, U12.C9 (DEVCLK-)
- new net SERDINA+: U12.T11 (SERDINA+)
- new net SERDINA-: U12.T10 (SERDINA-)
- new net SERDINB+: U12.U12 (SERDINB+)
- new net SERDINB-: U12.U13 (SERDINB-)
- new net SERDINC+: U12.T15 (SERDINC+)
- new net SERDINC-: U12.T14 (SERDINC-)
- new net SERDIND+: U12.U16 (SERDIND+)
- new net SERDIND-: U12.U17 (SERDIND-)
- new net SERDOUTA+: C425.1, C425.2, U12.T7 (SERDOUTA+)
- new net SERDOUTA-: C426.1, C426.2, U12.T8 (SERDOUTA-)
- new net SERDOUTB+: C427.1, C427.2, U12.U5 (SERDOUTB+)
- new net SERDOUTB-: C428.1, C428.2, U12.U6 (SERDOUTB-)
- new net SERDOUTC+: C429.1, C429.2, U12.T3 (SERDOUTC+)
- new net SERDOUTC-: C430.1, C430.2, U12.T4 (SERDOUTC-)
- new net SERDOUTD+: C431.1, C431.2, U12.U1 (SERDOUTD+)
- new net SERDOUTD-: C432.1, C432.2, U12.U2 (SERDOUTD-)
- new net SYNCIN1+: U12.N12 (SYNCIN1+)
- new net SYNCIN1-: U12.N13 (SYNCIN1-)
- new net SYNCIN2+: U12.P7 (SYNCIN2+)
- new net SYNCIN2-: U12.P8 (SYNCIN2-)
- new net SYNCIN3+: U12.N6 (SYNCIN3+)
- new net SYNCIN3-: U12.P6 (SYNCIN3-)
- new net SYNCOUT1+: U12.P15 (SYNCOUT1+)
- new net SYNCOUT1-: U12.R15 (SYNCOUT1-)
- new net SYNCOUT2+: U12.N14 (SYNCOUT2+)
- new net SYNCOUT2-: U12.N15 (SYNCOUT2-)
- new net SYSREF+: U12.D8 (SYSREF+)
- new net SYSREF-: U12.D9 (SYSREF-)
Other:
- removed sheet RF_Power_CFG
- removed sheet RF_SERDES
