File: RX_PATH.kicad_sch (KiCad schematic)
At the start: 0 parts

Commit message: pushing the schematics works
Parts:
- added C475, C480, C485, C486, C487, C488, C489, C490: 0.2p, Capacitor_SMD:C_0201_0603Metric, symbol Device:C
- added C476, C477, C478, C479, C481, C482, C483, C484: 3.9p, Capacitor_SMD:C_0201_0603Metric, symbol Device:C
- added C515, C516, C517, C518, C519, C520, C521, C522: 0.5p, Capacitor_SMD:C_0201_0603Metric, symbol Device:C
- added J10, J5, J8, J9: SMA_Edge_4.8MM, Connector_Coaxial:SMA_Samtec_SMA-J-P-H-ST-EM1_EdgeMount, symbol Connector:Conn_Coaxial_Small
- added L10, L21: 91n, Inductor_SMD:L_0201_0603Metric, symbol Device:L
- added L11, L20: 100n, Inductor_SMD:L_0201_0603Metric, symbol Device:L
- added L12, L23: 47n, Inductor_SMD:L_0201_0603Metric, symbol Device:L
- added L19, L22: 43n, Inductor_SMD:L_0201_0603Metric, symbol Device:L
- added R91, R92, R93, R94, R95, R96, R97, R98: 0, Resistor_SMD:R_0201_0603Metric, symbol Device:R
- added T5, T6, T7, T8: H3-TCM2-63WX+, dfdtc_RF:HT_TCP_2_25P, symbol dfdtc_RF:H3-TCM2-63WX+
Connections:
- new net: C480.1, R91.2, R95.1
- new net: R95.2, T5.3 (Port1)
- new net: C478.1, C519.1, L11.1, T6.6 (OUT+)
- new net: C479.1, C520.1, L11.2, T6.4 (OUT-)
- new net: C489.1, J9.1 (In), R93.1
- new net: C485.1, R93.2, R97.1
- new net: C477.1, C516.1, L10.2, T5.4 (OUT-)
- new net: C476.1, C515.1, L10.1, T5.6 (OUT+)
- new net: C482.1, C522.1, L20.2, T7.4 (OUT-)
- new net: R97.2, T7.3 (Port1)
- new net: R98.2, T8.3 (Port1)
- new net: C484.1, C518.1, L21.2, T8.4 (OUT-)
- new net: C483.1, C517.1, L21.1, T8.6 (OUT+)
- new net: C490.1, J10.1 (In), R94.1
- new net: C481.1, C521.1, L20.1, T7.6 (OUT+)
- new net: C487.1, J5.1 (In), R91.1
- new net: R96.2, T6.3 (Port1)
- new net: C486.1, R94.2, R98.1
- new net: C475.1, R92.2, R96.1
- new net: C488.1, J8.1 (In), R92.1
- new net GND: C475.2, C480.2, C485.2, C486.2, C487.2, C488.2, C489.2, C490.2, C515.2, C516.2, C517.2, C518.2, C519.2, C520.2, C521.2, C522.2, J10.2 (Ext), J5.2 (Ext), J8.2 (Ext), J9.2 (Ext), T5.5 (NC), T5.[1,2] (GND), T6.5 (NC), T6.[1,2] (GND), T7.5 (NC), T7.[1,2] (GND), T8.5 (NC), T8.[1,2] (GND)
- new net RX1+: C476.2, L12.1
- new net RX1-: C477.2, L12.2
- new net RX2+: C478.2, L19.1
- new net RX2-: C479.2, L19.2
- new net RX3+: C481.2, L22.1
- new net RX3-: C482.2, L22.2
- new net RX4+: C483.2, L23.1
- new net RX4-: C484.2, L23.2
