File: SYS_CLK.kicad_sch (KiCad schematic)
At the start: 14 parts, among them U13 AD9528BCPZ, Y1 NV0914BH3I155D30N122.88, Y2 OC5SC25

Commit message: pushing the schematics works
Parts:
- added C433, C434, C435, C436, C437, C438, C443, C444, C446, C447, C448, C449, C450, C451, C452, C453, C454, C455, C456, C457, C458, C459, C460, C461, C462, C463, C464, C465, C466, C544, C545, C546, C547: 100n, Capacitor_SMD:C_0201_0603Metric, symbol Device:C
- added C439, C440, C441, C442, C543: 10n C0G, Capacitor_SMD:C_0402_1005Metric, symbol Device:C
- added C445: 1.6n, Capacitor_SMD:C_0805_2012Metric, symbol Device:C
- added D4: ESD131-B1-W0201, Diode_SMD:Infineon_SG-WLL-2-3_0.58x0.28_P0.36mm, symbol Diode:ESD131-B1-W0201
- added IC6: LMK1C1102, dfdtc_SON:WSON-8_2x2mm_P0.5mm, symbol dfdtc_buffer:LMK1C1102
- added J4, J7: IPEX_G1, Connector_Coaxial:U.FL_Hirose_U.FL-R-SMT-1_Vertical, symbol Connector:Conn_Coaxial
- added R88, R89: 100, Resistor_SMD:R_0603_1608Metric, symbol Device:R
- C380: value 1n -> 680p
- C382: value 1u -> 15n
- C385: value 0.1u -> 300n; footprint Capacitor_SMD:C_0201_0603Metric -> Capacitor_SMD:C_0603_1608Metric
- R80: value 10.2k -> 3.09M
- R83: value R -> 50
- Y1: footprint dfdtc_VCO:Oscillator_SMD_Abracon_ABLNO_MOD -> Oscillator:Oscillator_SMD_Abracon_ABLNO
Connections:
- net 3V3: now also U13.1 (VDD), U13.10 (VDD), U13.16 (VDD), U13.20 (VDD), U13.27 (VDD13), U13.30 (VDD12), U13.33 (VDD11), U13.36 (VDD10), U13.39 (VDD9), U13.42 (VDD8), U13.45 (VDD7), U13.48 (VDD6), U13.51 (VDD5), U13.54 (VDD4), U13.60 (VDD3), U13.63 (VDD2), U13.66 (VDD1), U13.69 (VDD0), U13.72 (VDD), C438.2, C446.2, C447.2, C448.2, C449.2, C450.2, C451.2, C452.2, C453.2, C454.2, C455.2, C456.2, C457.2, C458.2, C459.2, C460.2, C461.2, C462.2, C463.2, C464.2, IC6.2 (1G), IC6.6 (VDD)
- net GND: now also R83.2, U13.57 (SYSREF_REQ), Y2.4 (GND), C437.1, C438.1, C442.2, C443.1, C444.1, C445.2, C446.1, C447.1, C448.1, C449.1, C450.1, C451.1, C452.1, C453.1, C454.1, C455.1, C456.1, C457.1, C458.1, C459.1, C460.1, C461.1, C462.1, C463.1, C464.1, C543.2, D4.1 (A1), IC6.4 (GND), J4.2 (Ext), J7.2 (Ext), R89.2
- net REFA+: now also C440.2
- net REFA-: now also C442.1
- net REFB+: now also D4.2 (A2), J7.1 (In)
- net REFB-: now also C543.1
- net at C382.1, R80.2: now also C445.1
- net +5V: now reaches Y2.2 (5V)
- net +5V: now also C437.2
- net at Y2.3 (RF): now also R83.1, C439.1
- net at Y2.5 (Uin): now also J4.1 (In)
- net ~{CLK_RESET}: now reaches U13.19 (*RESET)
- net CLK_GEN_CS: now reaches U13.21 (CS)
- net SCLK/SCL: now reaches U13.22 (SCLK/SCL)
- net SDIO/SDA: now reaches U13.23 (SDIO/SDA)
- net SDO: now reaches U13.24 (SDO)
- net OUT6+: now reaches U13.46 (OUT6+)
- net OUT6+: now also C546.1
- net OUT6-: now reaches U13.47 (OUT6-)
- net OUT6-: now also C547.1
- net OUT5+: now reaches U13.49 (OUT5+)
- net OUT5+: now also C544.1
- net OUT5-: now reaches U13.50 (OUT5-)
- net OUT5-: now also C545.1
- net OUT4+: now reaches U13.52 (OUT4+)
- net OUT4+: now also C465.1
- net OUT4-: now reaches U13.53 (OUT4-)
- net OUT4-: now also C466.1
- net STATUS0/SP0: now reaches U13.55 (STATUS0/SP0)
- net STATUS1/SP1: now reaches U13.56 (STATUS1/SP1)
- net FPGA_SYSREF+: now reaches U13.58 (OUT3+)
- net FPGA_SYSREF-: now reaches U13.59 (OUT3-)
- net OUT2+: now reaches U13.61 (OUT2+)
- net OUT2+: now also C435.1
- net OUT2-: now reaches U13.62 (OUT2-)
- net OUT2-: now also C436.1
- net SYSREF+: now reaches U13.64 (OUT1+)
- net SYSREF-: now reaches U13.65 (OUT1-)
- net OUT0+: now reaches U13.67 (OUT0+)
- net OUT0+: now also C433.1
- net OUT0-: now reaches U13.68 (OUT0-)
- net OUT0-: now also C434.1
- net at U13.70 (SYSREF_IN+): now also C443.2
- net at U13.71 (SYSREF_IN-): now also C444.2
- new net: C439.2, IC6.1 (CLKIN), R88.2, R89.1
- new net: C440.1, IC6.3 (Y0)
- new net: IC6.5 (NC), IC6.7 (NC)
- new net: C441.1, IC6.8 (Y1)
- new net +3V3: R88.1
- new net D4_SYS_CLK_N: C547.2
- new net D4_SYS_CLK_P: C546.2
- new net DEVCLK+: C433.2
- new net DEVCLK-: C434.2
- new net DEVCLK1+: C544.2
- new net DEVCLK1-: C545.2
- new net FPGA_DEVCLK+: C435.2
- new net FPGA_DEVCLK-: C436.2
- new net GTY_DEVCLK+: C465.2
- new net GTY_DEVCLK-: C466.2
- no-connect marks 0 -> 16
Other:
- moved on the sheet: C381, C382, R80, R83, U13B, Y2
