File: TX_PATH.kicad_sch (KiCad schematic)
At the start: 0 parts

Commit message: pushing the schematics works
Parts:
- added C491, C492, C493, C494, C495, C496, C497, C498, C523, C524, C525, C526, C527, C528, C529, C530: 0.2p, Capacitor_SMD:C_0201_0603Metric, symbol Device:C
- added C499, C500, C503, C504: 10p, Capacitor_SMD:C_0201_0603Metric, symbol Device:C
- added C501, C502, C505, C506: 4.7p, Capacitor_SMD:C_0201_0603Metric, symbol Device:C
- added C507, C508, C509, C510, C511, C512, C513, C514: 0.5p, Capacitor_SMD:C_0201_0603Metric, symbol Device:C
- added J11, J12, J13, J14: SMA_Edge_4.8MM, Connector_Coaxial:SMA_Samtec_SMA-J-P-H-ST-EM1_EdgeMount, symbol Connector:Conn_Coaxial_Small
- added J15, J16, J17, J18: IPEX_G1, Connector_Coaxial:U.FL_Hirose_U.FL-R-SMT-1_Vertical, symbol Connector:Conn_Coaxial_Small
- added L1, L7: 100n, symbol Device:L
- added L2, L8: 47n, symbol Device:L
- added L24, L26, L28, L30: 200n, Inductor_SMD:L_0201_0603Metric, symbol Device:L
- added L25, L27: 82n, Inductor_SMD:L_0201_0603Metric, symbol Device:L
- added L29, L31: 75n, Inductor_SMD:L_0201_0603Metric, symbol Device:L
- added L3, L5: 91n, symbol Device:L
- added L32, L34: 0.9n, Inductor_SMD:L_0201_0603Metric, symbol Device:L
- added L33, L35: 0.8n, Inductor_SMD:L_0201_0603Metric, symbol Device:L
- added L4, L6: 43n, symbol Device:L
- added R100, R101, R102, R103, R104, R105, R106, R107, R108, R109, R110, R111, R112, R113, R114, R115, R116, R117, R118, R99: 0, Resistor_SMD:R_0201_0603Metric, symbol Device:R
- added T10, T11, T12, T9: ETC1-1-13TR, dfdtc_RF:HT_TCP_2_25P, symbol dfdtc_RF:ETC1-1-13TR
- added T13, T14, T15, T16: H3-TCM2-63WX+, dfdtc_RF:HT_TCP_2_25P, symbol dfdtc_RF:H3-TCM2-63WX+
Connections:
- new net: C491.1, J15.1 (In), R99.1
- new net: L33.2, T9.1 (IN)
- new net: L5.2, R110.1, T9.4 (OUT-)
- new net: L5.1, R109.1, T9.6 (OUT+)
- new net: C497.1, R101.2, R105.1
- new net: R105.2, T15.3 (Port1)
- new net: C525.1, J12.1 (In), R116.1
- new net: L3.2, R114.1, T12.4 (OUT-)
- new net: C527.1, J13.1 (In), R117.1
- new net: C496.1, R100.2, R104.1
- new net: R104.2, T14.3 (Port1)
- new net: C492.1, J16.1 (In), R100.1
- new net: C504.1, C512.1, L26.2, T15.4 (OUT-)
- new net: C503.1, C511.1, L26.1, T15.6 (OUT+)
- new net: C530.1, L35.1, R118.2
- new net: C501.1, C508.1, L25.1, T14.6 (OUT+)
- new net: R106.2, T16.3 (Port1)
- new net: C506.1, C510.1, L27.2, T16.4 (OUT-)
- new net: C505.1, C509.1, L27.1, T16.6 (OUT+)
- new net: C495.1, R103.1, R99.2
- new net: C502.1, C507.1, L25.2, T14.4 (OUT-)
- new net: C526.1, L32.1, R116.2
- new net: L1.2, R112.1, T11.4 (OUT-)
- new net: R103.2, T13.3 (Port1)
- new net: C500.1, C514.1, L24.2, T13.4 (OUT-)
- new net: C499.1, C513.1, L24.1, T13.6 (OUT+)
- new net: L35.2, T12.1 (IN)
- new net: L3.1, R113.1, T12.6 (OUT+)
- new net: C494.1, J18.1 (In), R102.1
- new net: C523.1, J11.1 (In), R115.1
- new net: C524.1, L33.1, R115.2
- new net: C493.1, J17.1 (In), R101.1
- new net: L32.2, T10.1 (IN)
- new net: L7.2, R108.1, T10.4 (OUT-)
- new net: L7.1, R107.1, T10.6 (OUT+)
- new net: C528.1, L34.1, R117.2
- new net: C529.1, J14.1 (In), R118.1
- new net: C498.1, R102.2, R106.1
- new net: L1.1, R111.1, T11.6 (OUT+)
- new net: L34.2, T11.1 (IN)
- new net GND: C491.2, C492.2, C493.2, C494.2, C495.2, C496.2, C497.2, C498.2, C507.2, C508.2, C509.2, C510.2, C511.2, C512.2, C513.2, C514.2, C523.2, C524.2, C525.2, C526.2, C527.2, C528.2, C529.2, C530.2, J11.2 (Ext), J12.2 (Ext), J13.2 (Ext), J14.2 (Ext), J15.2 (Ext), J16.2 (Ext), J17.2 (Ext), J18.2 (Ext), T10.2 (NC), T10.3 (GND), T10.5 (GND), T11.2 (NC), T11.3 (GND), T11.5 (GND), T12.2 (NC), T12.3 (GND), T12.5 (GND), T13.5 (NC), T13.[1,2] (GND), T14.5 (NC), T14.[1,2] (GND), T15.5 (NC), T15.[1,2] (GND), T16.5 (NC), T16.[1,2] (GND), T9.2 (NC), T9.3 (GND), T9.5 (GND)
- new net ORX1+: C499.2, L28.1
- new net ORX1-: C500.2, L28.2
- new net ORX2+: C501.2, L29.1
- new net ORX2-: C502.2, L29.2
- new net ORX3+: C503.2, L30.1
- new net ORX3-: C504.2, L30.2
- new net ORX4+: C505.2, L31.1
- new net ORX4-: C506.2, L31.2
- new net TX1+: L8.1, R109.2
- new net TX1-: L8.2, R110.2
- new net TX2+: L6.1, R107.2
- new net TX2-: L6.2, R108.2
- new net TX3+: L4.1, R111.2
- new net TX3-: L4.2, R112.2
- new net TX4+: L2.1, R113.2
- new net TX4-: L2.2, R114.2
Other:
- note added: "CH1"
- note added: "CH2"
- note added: "CH3"
- note added: "CH4"
