File: VCCINT.kicad_sch (KiCad schematic)
At the start: 88 parts

Commit message: pushing the schematics works
Parts:
- C1, C2, C60, C62, C64, C66: value C_Polarized -> 100u
- C10, C4, C6, C8: value C -> 4.7u
- C11, C12, C13, C14, C15, C16, C17, C18: value C -> 2.2u
- C19, C20, C21, C22, C23, C24, C25, C26, C27, C28, C29, C30, C31, C32, C33, C34, C35, C36, C37, C38, C39, C40, C41, C42, C43, C44, C45, C46, C47, C48, C49, C50, C51, C52, C53, C54, C55, C56, C57, C58, C59, C61, C63, C65: value C -> 22u
- C3, C5, C7, C9: value C -> 100n
- C67, C68, C69, C70, C71, C72: value C -> 1u
- R1, R2: value R -> 91K
- R10, R7: value R -> 49.9K
- R11: value R -> 80.6K
- R12, R8: value R -> 30K
- R3, R4, R9: value R -> 20K
- R5, R6: value R -> 10K
